Commit message: Fixed missing param

File: fitzroy_description/urdf/fitzroy.urdf.xacro (robot description, xacro)
@@ -62,4 +62,5 @@
   <!-- Sensor Locations -->
   <xacro:property name="gps_y" value="-0.02"/>
+  <xacro:property name="ranger_size" value="0.01"/>
 	<!-- default initializer for inertia -->
 	<xacro:macro name="default_inertial" params="mass">
@@ -122,38 +123,8 @@
 	<!-- base footprint to make everything work better -->
   <link name="base_footprint">
-    <visual>
-      <geometry>
-        <box size="0.001 0.001 0.001"/>
-      </geometry>
-			<origin rpy="0 0 0" xyz="0 0 0"/>
-			<material name="white"/>
-    </visual>
-		<inertial>
-			<mass value="0.0001"/>
-			<origin xyz="0 0 0"/>
-			<inertia ixx="0.0001" ixy="0.0" ixz="0.0" iyy="0.0001" iyz="0.0" izz="0.0001"/>
-		</inertial>
-  </link>
-	<gazebo reference="base_footprint">
-		<material>Gazebo/White</material>
-	</gazebo>
+  </link>
 	<!-- base link for whole car ${wheelbase/2} -->
   <link name="base_link">
-    <visual>
-      <geometry>
-        <box size="0.001 0.001 0.001"/>
-      </geometry>
-			<material name="white"/>
-    </visual>
-		<collision>
-			<geometry>
-				<box size="0.001 0.001 0.001"/>
-			</geometry>
-		</collision>
-		<xacro:default_inertial mass="1"/>
-  </link>
-	<gazebo reference="base_link">
-		<material>Gazebo/White</material>
-	</gazebo>
+  </link>
 	<joint name="base_footprint_to_base_link" type="fixed">
     <parent link="base_footprint"/>
@@ -183,5 +154,5 @@
     <parent link="base_link"/>
     <child link="chassis"/>
-    <origin xyz="0 0 ${chasisheight/2 + rear_shock_offset} "/>
+    <origin xyz="0 0 ${rear_shock_offset} "/>
   </joint>
 	<!-- rear axle -->
@@ -503,5 +474,5 @@
 		<collision>
 			<geometry>
-				<box size="${framewidth} ${frameheight} ${thickness}"/>
+        <box size="${frameheight} ${framewidth} ${thickness}"/>
 			</geometry>
 			<!-- <origin rpy="0 ${pi/2} 0" xyz="0 0 ${-chasisheight/2} "/> -->

Commit message: Added ultrasonic

File: fitzroy_description/urdf/fitzroy.urdf.xacro (robot description, xacro)
@@ -2,7 +2,5 @@
 <robot xmlns:xacro="http://www.ros.org/wiki/xacro" name="fitzroy">
 	<!-- roslaunch urdf_tutorial xacrodisplay.launch model:='$(find fitzroy_description)/urdf/tractorcustom.urdf.xacro' gui:='true'-->
-	<!-- Each link is a physical element, the visual tag is required -->
-	<!-- Each link also has a collision and inertial element which define interactions -->
-	<xacro:property name="pi" value="3.14159265358" />
+  <xacro:include filename="$(find fitzroy_description)/urdf/fitzroy_common.urdf.xacro"/>
   <!-- The fake GPS needs an origin, it's an arg so it can be changed based on the world used. -->
   <!-- This is the origin of the gazebo world, NOT the place the robot is first dropped into. -->
@@ -63,62 +61,4 @@
   <xacro:property name="gps_y" value="-0.02"/>
   <xacro:property name="ranger_size" value="0.01"/>
-	<!-- default initializer for inertia -->
-	<xacro:macro name="default_inertial" params="mass">
-		<inertial>
-      			<mass value="${mass}" />
-		        <inertia ixx="1.0" ixy="0.0" ixz="0.0"
-			         iyy="1.0" iyz="0.0"
-			         izz="1.0" />
-		</inertial>
-	</xacro:macro>
-	<!-- macro for computing the inertia tensor for cubes-->
-	<!-- https://en.wikipedia.org/wiki/List_of_moments_of_inertia -->
-	<xacro:macro name="cube_inertial"
-               params="dimx dimy dimz mass">
-    <inertial>
-      <mass value="${mass}"/>
-      <inertia ixx="${(1/12)*mass*(dimy*dimy + dimz*dimz)}"
-               ixy="0" ixz="0"
-               iyy="${(1/12)*mass*(dimx*dimx + dimz*dimz)}"
-               iyz="0"
-               izz="${(1/12)*mass*(dimx*dimx + dimy*dimy)}"/>
-    </inertial>
-  </xacro:macro>
-	<!-- macro for computing inertia tensor for a cylinder-->
-	<!-- http://scienceworld.wolfram.com/physics/MomentofInertiaCylinder.html -->
-	<xacro:macro name="cylinder_inertial"
-               params="rad height mass">
-    <inertial>
-      <mass value="${mass}"/>
-      <inertia ixx="${(1/12)*mass*(height*height) + (1 / 4)*mass*(rad*rad) }"
-               ixy="0" ixz="0"
-               iyy="${(1/12)*mass*(height*height) + (1 / 4)*mass*(rad*rad) }"
-               iyz="0"
-               izz="${(1/2)* mass * (rad*rad)}"/>
-    </inertial>
-  </xacro:macro>
-	<!-- Setup some colors -->
-	<!-- List of materials: http://wiki.ros.org/simulator_gazebo/Tutorials/ListOfMaterials-->
-	<material name="blue">
-		<color rgba="0 0 0.8 1"/>
-	</material>
-	<material name="red">
-		<color rgba="0.8 0 0 1"/>
-	</material>
-	<material name="hideaxle">
-		<color rgba="1 1 1 1"/>
-	</material>
-	<material name="white">
-		<color rgba="1 1 1 1"/>
-	</material>
-	<material name="black">
-		<color rgba="0 0 0 1"/>
-	</material>
-	<material name="grey">
-		<color rgba="0.3 0.3 0.3 1"/>
-	</material>
-	<material name="green">
-		<color rgba="0 0.6 0 1"/>
-	</material>
 	<!-- base footprint to make everything work better -->
   <link name="base_footprint">
@@ -157,22 +97,9 @@
   </joint>
 	<!-- rear axle -->
-  <link name="rear_axle">
-    <visual>
-      <geometry>
-        <box size="${axlesize} ${rearwheelsep-rearwheelwidth} ${axlesize}"/>
-      </geometry>
-			<origin rpy="0 0 0" xyz="0 0 0"/>
-			<material name="hideaxle"/>
-    </visual>
-		<collision>
-			<geometry>
-				<box size="${axlesize} ${rearwheelsep-rearwheelwidth} ${axlesize}"/>
-			</geometry>
-		</collision>
-		<xacro:default_inertial mass="10"/>
-  </link>
-	<gazebo reference="rear_axle">
-		<material>Gazebo/White</material>
-	</gazebo>
+	<xacro:cube_aluminum
+      name="rear_axle"
+      dimx="${axlesize}"
+      dimy="${rearwheelsep-rearwheelwidth}"
+      dimz="${axlesize}" />
 	<joint name="base_link_to_rear_axle" type="fixed">
     <parent link="chassis"/>
@@ -751,3 +678,8 @@
     <origin xyz="${-(wheelbase/2 + rackback)} 0 ${rackheight}" rpy="0 0 0"/>
   </picam>
+	<!-- Ultrasonic -->
+  <xacro:include filename="$(find fitzroy_description)/urdf/ultrasonic_sensor.urdf.xacro"/>
+  <ultrasonic_sensor parent="base_link" name="ultrasonic">
+    <origin xyz="${-(wheelbase/2 + rackback)} 0.020 ${rackheight}" rpy="0 0 0"/>
+  </ultrasonic_sensor>
 </robot>

Commit message: Still wonky in gazebo

File: fitzroy_description/urdf/fitzroy.urdf.xacro (robot description, xacro)
@@ -10,5 +10,5 @@
 	<!-- Front Loader Properties-->
 	<xacro:property name="framewidth" value="0.07" />
-	<xacro:property name="frameheight" value="0.1" />
+	<xacro:property name="frameheight" value="0.05" />
 	<xacro:property name="thickness" value="0.01" />
 	<xacro:property name="armsize" value="0.01" />
@@ -31,5 +31,5 @@
 	<xacro:property name="chasismass" value="0.25"/>
 	<!-- Backrack on tractor that Reed made-->
-	<xacro:property name="rackheight" value="0.19" />
+	<xacro:property name="rackheight" value="0.09" />
 	<xacro:property name="rackback" value="-0.015" />
 	<!-- Wheel properties-->
@@ -73,22 +73,9 @@
   </joint>
 	<!-- main chasis -->
-  <link name="chassis">
-    <visual>
-      <geometry>
-        <box size="${chasislength} ${chasiswidth} ${chasisheight}"/>
-      </geometry>
-    </visual>
-		<collision> <!-- this defines the collision shape (usually same as visual shape)-->
-			<geometry>
-        <box size="${chasislength} ${chasiswidth} ${chasisheight}"/>
-			</geometry>
-		</collision>
-		<xacro:cube_inertial
-        dimx="${chasislength}" dimy="${chasiswidth}"
-        dimz="${chasisheight}" mass="${chasismass}" />
-  </link>
-	<!-- <gazebo reference="chassis">
-		<material>Gazebo/Green</material>
-	</gazebo> -->
+	<xacro:cube_plastic
+      name="chassis"
+      dimx="${chasislength}"
+      dimy="${chasiswidth}"
+      dimz="${chasisheight}" />
 	<joint name="base_link_to_chasis" type="fixed">
     <parent link="base_link"/>
@@ -373,50 +360,50 @@
     <mimic  joint="back_to_left_arm" multiplier="1" offset="0"/>
   </joint>
-	<!-- front grate -->
-  <link name="front_grate">
-    <visual>
-      <geometry>
-        <box size="${frameheight} ${framewidth} ${thickness}"/>
-      </geometry>
-			<!-- <origin rpy="0 ${pi/2} 0" xyz="0 0 ${-chasisheight/2} "/> -->
-			<origin rpy="0 ${pi/2} 0" xyz="${frame_x} 0 ${chasisheight-frame_z} "/>
-			<material name="grey"/>
-    </visual>
-    <visual>
-      <geometry>
-        <box size="${forkheight} ${forkwidth} ${forklen}"/>
-      </geometry>
-			<!-- <origin rpy="0 ${pi/2} 0" xyz="0 0 ${-chasisheight/2} "/> -->
-			<origin rpy="0 ${pi/2} 0" xyz="${frame_x+forklen/2} ${forksep/2} ${chasisheight-frame_z-frameheight/2} "/>
-			<material name="grey"/>
-    </visual>
-    <visual>
-      <geometry>
-        <box size="${forkheight} ${forkwidth} ${forklen}"/>
-      </geometry>
-			<!-- <origin rpy="0 ${pi/2} 0" xyz="0 0 ${-chasisheight/2} "/> -->
-			<origin rpy="0 ${pi/2} 0" xyz="${frame_x+forklen/2} ${-forksep/2} ${chasisheight-frame_z-frameheight/2} "/>
-			<material name="grey"/>
-    </visual>
-		<collision>
-			<geometry>
-        <box size="${frameheight} ${framewidth} ${thickness}"/>
-			</geometry>
-			<!-- <origin rpy="0 ${pi/2} 0" xyz="0 0 ${-chasisheight/2} "/> -->
-			<origin rpy="0 ${pi/2} 0" xyz="${frame_x} 0 ${chasisheight-frame_z} "/>
-		</collision>
-		<xacro:default_inertial mass="1"/>
-  </link>
-	<gazebo reference="front_grate">
-		<material>Gazebo/DarkGrey</material>
-	</gazebo>
+	<!-- START OF FORK ASSEMBLY -->
+	<!-- We use separate links for each part to have accurate physics properties -->
+	<!-- fork assembly -->
+  <link name="fork_assembly">
+  </link>
 	<!-- lift front wall with arm -->
-	<joint name="left_arm_to_front_grate" type="revolute">
+	<joint name="left_arm_to_fork_assembly" type="revolute">
 		<axis xyz="0 -1 0"/>
     <limit effort="1000.0" lower="${liftmin}" upper="${liftmax}" velocity="0.5"/>
     <parent link="left_arm"/>
-    <child link="front_grate"/>
+    <child link="fork_assembly"/>
     <!-- <origin xyz="${armlen-thickness} ${-framewidth/2 - armsize/2} 0"/> -->
     <origin xyz="${armlen-thickness} ${-framewidth/2 + armsize/2} 0"/>
+  </joint>
+	<!-- backstop -->
+	<xacro:cube_aluminum
+      name="fork_backstop"
+      dimx="${frameheight}"
+      dimy="${framewidth}"
+      dimz="${thickness}" />
+	<joint name="fork_assembly_to_fork_backstop" type="fixed">
+    <parent link="fork_assembly"/>
+    <child link="fork_backstop"/>
+		<origin rpy="0 ${pi/2} 0" xyz="${frame_x} 0 ${chasisheight-frame_z} "/>
+  </joint>
+	<!-- left fork -->
+	<xacro:cube_aluminum
+      name="left_fork"
+      dimx="${forkheight}"
+      dimy="${forkwidth}"
+      dimz="${forklen}" />
+	<joint name="fork_assembly_to_left_fork" type="fixed">
+    <parent link="fork_assembly"/>
+    <child link="left_fork"/>
+    <origin rpy="0 ${pi/2} 0" xyz="${frame_x+forklen/2} ${ forksep/2} ${chasisheight-frame_z-frameheight/2} "/>
+  </joint>
+	<!-- right fork -->
+	<xacro:cube_aluminum
+      name="right_fork"
+      dimx="${forkheight}"
+      dimy="${forkwidth}"
+      dimz="${forklen}" />
+	<joint name="fork_assembly_to_right_fork" type="fixed">
+    <parent link="fork_assembly"/>
+    <child link="right_fork"/>
+    <origin rpy="0 ${pi/2} 0" xyz="${frame_x+forklen/2} ${-forksep/2} ${chasisheight-frame_z-frameheight/2} "/>
   </joint>
 	<!-- START OF THE TRANSMISSIONS STUFF (NECCESARY TO USE MOTOR CONTROL IN GAZEBO) -->
@@ -501,5 +488,5 @@
       <mechanicalReduction>1</mechanicalReduction>
     </actuator>
-    <joint name="left_arm_to_front_grate">
+    <joint name="left_arm_to_fork_assembly">
       <hardwareInterface>PositionJointInterface</hardwareInterface>
     </joint>
@@ -521,93 +508,11 @@
       <rpyOffsets>0 0 0</rpyOffsets>
     </plugin>
-	<plugin name="magnetic" filename="libhector_gazebo_ros_magnetic.so">
-		 <alwaysOn>1</alwaysOn>
-		 <updateRate>30.0</updateRate> <!-- make this the same rate as imu plugin -->
-		 <bodyName>imu_link</bodyName>
-			<frameId>mag_link</frameId> <!-- 'frameId' not 'frameName'-->
-		 <topicName>/imu/mag</topicName>
-	</plugin>
-  </gazebo>
-	<!-- Range finder out the back to sense for objects behind us -->
-	<joint name="radar_joint_back" type="fixed">
-    <origin xyz="${-chasislength/2-ranger_size/2} 0 ${-chasisheight/2}" rpy="0 0 ${pi}"/>
-    <parent link="chassis"/>
-    <child link="radar_link"/>
-  </joint>
-  <link name="radar_link">
-    <visual>
-      <geometry>
-        <box size="${ranger_size} ${ranger_size} ${ranger_size}"/>
-      </geometry>
-    </visual>
-    <inertial>
-      <mass value="1e-5" />
-      <origin xyz="0 0 0" rpy="0 0 0"/>
-      <inertia ixx="1e-6" ixy="0" ixz="0" iyy="1e-6" iyz="0" izz="1e-6" />
-    </inertial>
-  </link>
-	<gazebo reference="radar_link">
-     <sensor type="ray" name="rear_range">
-      <pose>0 0 0 0 0 0</pose>
-      <update_rate>30</update_rate>
-			<visualize>false</visualize>
-      <ray>
-          <scan>
-            <horizontal>
-              <samples>5</samples>
-              <resolution>1</resolution>
-              <min_angle>-0.2</min_angle>
-              <max_angle>0.2</max_angle>
-            </horizontal>
-            <vertical>
-              <samples>5</samples>
-              <resolution>1</resolution>
-              <min_angle>-0.01</min_angle>
-              <max_angle>0.01</max_angle>
-            </vertical>
-          </scan>
-          <range>
-            <min>0.01</min>
-            <max>5.0</max>
-            <resolution>0.01</resolution>
-          </range>
-			</ray>
-      <plugin name="gazebo_ros_rear_range" filename="libgazebo_ros_range.so">
-				<gaussianNoise>0.005</gaussianNoise>
-        <alwaysOn>true</alwaysOn>
-				<updateRate>30</updateRate>
-        <topicName>/back_up/radar</topicName>
-        <frameName>radar_link</frameName>
-				<fov>0.4</fov>
-				<radiation>ultrasound</radiation>
-      </plugin>
-    </sensor>
-		<material>Gazebo/Blue</material>
   </gazebo>
 	<!-- Setup a fake gps sensor -->
 	<joint name="gps_joint" type="fixed">
-    <axis xyz="1 0 0"/> <!-- 0 1 0 -->
-    <origin xyz="${-(wheelbase/2 + rackback)} ${gps_y} ${rackheight}"/>
     <parent link="base_link"/>
     <child link="gps_link"/>
   </joint>
 	<link name="gps_link">
-		<inertial>
-		  <mass value="0.001"/>
-		  <origin rpy="0 0 0" xyz="0 0 0"/>
-		  <inertia ixx="0.0001" ixy="0" ixz="0" iyy="0.000001" iyz="0" izz="0.0001"/>
-		</inertial>
-		<visual>
-		  <origin rpy="0 0 0" xyz="0 0 0"/>
-		  <geometry>
-		    <box size="0.001 0.001 0.001"/>
-		  </geometry>
-		</visual>
-		<collision>
-		  <origin rpy="0 0 0" xyz="0 0 0"/>
-		  <geometry>
-		    <box size=".001 .001 .001"/>
-		  </geometry>
-		</collision>
 	</link>
 	<gazebo>
@@ -630,27 +535,8 @@
 	<!-- Setup a fake IMU sensor -->
   <joint name="imu_joint" type="fixed">
-    <axis xyz="1 0 0"/> <!-- 0 1 0 -->
-    <origin xyz="-0.55 0.0 0.48 "/>
     <parent link="base_link"/>
     <child link="imu_link"/>
   </joint>
 	<link name="imu_link">
-		<inertial>
-		  <mass value="0.001"/>
-		  <origin rpy="0 0 0" xyz="0 0 0"/>
-		  <inertia ixx="0.0001" ixy="0" ixz="0" iyy="0.000001" iyz="0" izz="0.0001"/>
-		</inertial>
-		<visual>
-		  <origin rpy="0 0 0" xyz="0 0 0"/>
-		  <geometry>
-		    <box size="0.001 0.001 0.001"/>
-		  </geometry>
-		</visual>
-		<collision>
-		  <origin rpy="0 0 0" xyz="0 0 0"/>
-		  <geometry>
-		    <box size=".001 .001 .001"/>
-		  </geometry>
-		</collision>
 	</link>
 	<gazebo>
@@ -666,11 +552,4 @@
     </plugin>
 	</gazebo>
-<xacro:if value="$(arg use_velodyne)">
-	<!-- 3D LIDAR -->
-  <xacro:include filename="$(find velodyne_description)/urdf/HDL-32E.urdf.xacro"/>
-  <HDL-32E parent="base_link" name="velodyne" topic="/velodyne_points" hz="10" samples="900" noise="0.03" gpu="true">
-		<origin xyz="${-(wheelbase/2 + rackback)} 0.1 ${rackheight}" rpy="0 0 0"/>
-  </HDL-32E>
-</xacro:if>
 	<!-- Camera -->
   <xacro:include filename="$(find fitzroy_description)/urdf/picam.urdf.xacro"/>

File: fitzroy_description/urdf/fitzroy_common.urdf.xacro (robot description, xacro)
@@ -87,3 +87,27 @@
 	  </gazebo>
   </xacro:macro>
+	<!-- macro for creating a plastic cube -->
+	<xacro:macro name="cube_plastic"
+               params="name dimx dimy dimz density:=1000">
+    <xacro:property name="mass" value="${density*dimx*dimy*dimz}"/>
+    <link name="${name}">
+      <visual>
+        <geometry>
+          <box size="${dimx} ${dimy} ${dimz}"/>
+        </geometry>
+			  <origin rpy="0 0 0" xyz="0 0 0"/>
+			  <material name="red"/>
+      </visual>
+		  <collision>
+        <geometry>
+          <box size="${dimx} ${dimy} ${dimz}"/>
+        </geometry>
+			  <origin rpy="0 0 0" xyz="0 0 0"/>
+		  </collision>
+      <cube_inertial dimx="${dimx}" dimy="${dimy}" dimz="${dimz}" mass="${mass}" />
+    </link>
+	  <gazebo reference="${name}">
+		  <material>Gazebo/Red</material>
+	  </gazebo>
+  </xacro:macro>
 </robot>

File: fitzroy_description/urdf/picam.urdf.xacro (robot description, xacro)
@@ -10,5 +10,4 @@
 	<joint name="${name}_joint" type="fixed">
     <xacro:insert_block name="origin" />
-    <axis xyz="0 1 0" />
     <parent link="${parent}"/>
     <child link="${name}_link"/>

Commit message: Fixed crazy physics problem The front axles were 10kg!

File: fitzroy_description/urdf/fitzroy.urdf.xacro (robot description, xacro)
@@ -161,22 +161,9 @@
   </joint>
 	<!-- front axle right -->
-  <link name="front_axle_right">
-    <visual>
-      <geometry>
-        <box size="${axlesize} ${axlesize} ${axlesize}"/>
-      </geometry>
-			<origin rpy="0 0 0" xyz="0 0 0"/>
-			<material name="hideaxle"/>
-    </visual>
-		<collision>
-			<geometry>
-				<box size="${axlesize} ${axlesize} ${axlesize}"/>
-			</geometry>
-		</collision>
-		<xacro:default_inertial mass="10"/>
-  </link>
-	<gazebo reference="front_axle_right">
-		<material>Gazebo/White</material>
-	</gazebo>
+	<xacro:cube_aluminum
+      name="front_axle_right"
+      dimx="${axlesize}"
+      dimy="${axlesize}"
+      dimz="${axlesize}" />
 	<joint name="base_link_to_front_axle_right" type="revolute">
 		<axis xyz="0 0 1"/>
@@ -187,22 +174,9 @@
   </joint>
 	<!-- front axle left -->
-	<link name="front_axle_left">
-    <visual>
-      <geometry>
-        <box size="${axlesize} ${axlesize} ${axlesize}"/>
-      </geometry>
-			<origin rpy="0 0 0" xyz="0 0 0"/>
-			<material name="hideaxle"/>
-    </visual>
-		<collision>
-			<geometry>
-				<box size="${axlesize} ${axlesize} ${axlesize}"/>
-			</geometry>
-		</collision>
-		<xacro:default_inertial mass="10"/>
-  </link>
-	<gazebo reference="front_axle_left">
-		<material>Gazebo/White</material>
-	</gazebo>
+	<xacro:cube_aluminum
+      name="front_axle_left"
+      dimx="${axlesize}"
+      dimy="${axlesize}"
+      dimz="${axlesize}" />
 	<joint name="base_link_to_front_axle_left" type="revolute">
 		<axis xyz="0 0 1"/>
@@ -415,5 +389,5 @@
     </actuator>
     <joint name="base_link_to_front_axle_right">
-      <hardwareInterface>PositionJointInterface</hardwareInterface>
+      <hardwareInterface>hardware_interface/PositionJointInterface</hardwareInterface>
     </joint>
   </transmission>
@@ -424,5 +398,5 @@
     </actuator>
     <joint name="base_link_to_front_axle_left">
-      <hardwareInterface>PositionJointInterface</hardwareInterface>
+      <hardwareInterface>hardware_interface/PositionJointInterface</hardwareInterface>
     </joint>
   </transmission>
@@ -434,5 +408,5 @@
     </actuator>
     <joint name="front_axle_to_right_wheel">
-      <hardwareInterface>EffortJointInterface</hardwareInterface>
+      <hardwareInterface>hardware_interface/EffortJointInterface</hardwareInterface>
     </joint>
   </transmission>
@@ -443,5 +417,5 @@
     </actuator>
     <joint name="rear_axle_to_right_wheel">
-      <hardwareInterface>EffortJointInterface</hardwareInterface>
+      <hardwareInterface>hardware_interface/EffortJointInterface</hardwareInterface>
     </joint>
   </transmission>
@@ -452,5 +426,5 @@
     </actuator>
     <joint name="front_axle_to_left_wheel">
-      <hardwareInterface>EffortJointInterface</hardwareInterface>
+      <hardwareInterface>hardware_interface/EffortJointInterface</hardwareInterface>
     </joint>
   </transmission>
@@ -461,5 +435,5 @@
     </actuator>
     <joint name="rear_axle_to_left_wheel">
-      <hardwareInterface>EffortJointInterface</hardwareInterface>
+      <hardwareInterface>hardware_interface/EffortJointInterface</hardwareInterface>
     </joint>
   </transmission>
@@ -471,5 +445,5 @@
     </actuator>
     <joint name="back_to_left_arm">
-      <hardwareInterface>PositionJointInterface</hardwareInterface>
+      <hardwareInterface>hardware_interface/PositionJointInterface</hardwareInterface>
     </joint>
   </transmission>
@@ -480,5 +454,5 @@
     </actuator>
     <joint name="back_to_right_arm">
-      <hardwareInterface>PositionJointInterface</hardwareInterface>
+      <hardwareInterface>hardware_interface/PositionJointInterface</hardwareInterface>
     </joint>
   </transmission>
@@ -489,5 +463,5 @@
     </actuator>
     <joint name="left_arm_to_fork_assembly">
-      <hardwareInterface>PositionJointInterface</hardwareInterface>
+      <hardwareInterface>hardware_interface/PositionJointInterface</hardwareInterface>
     </joint>
   </transmission>
@@ -495,5 +469,7 @@
 	<gazebo>
     <plugin name="gazebo_ros_control" filename="libgazebo_ros_control.so">
-      <robotNamespace>/</robotNamespace>
+      <robotNamespace>/fitzroy</robotNamespace>
+      <robotSimType>gazebo_ros_control/DefaultRobotHWSim</robotSimType>
+      <legacyModeNS>true</legacyModeNS>
     </plugin>
 	<!-- Provide pose as an odom topic -->

File: fitzroy_description/urdf/picam.urdf.xacro (robot description, xacro)
@@ -16,5 +16,5 @@
     <collision>
       <geometry>
-    		<box size="${picam_thickness} ${picam_width} ${picam_height} "/>
+    	  <box size="${picam_thickness} ${picam_width} ${picam_height} "/>
       </geometry>
     </collision>
