Commit message: two steps forward... two steps back.

File: fitzroy_description/urdf/fitzroy.urdf.xacro (robot description, xacro)
@@ -70,5 +70,5 @@
     <parent link="base_footprint"/>
     <child link="base_link"/>
-    <origin xyz="${wheelbase/2} 0 ${rearwheeldia/2} "/>
+    <origin xyz="0 0 ${rearwheeldia/2} "/>
   </joint>
 	<!-- main chasis -->
@@ -81,5 +81,5 @@
     <parent link="base_link"/>
     <child link="chassis"/>
-    <origin xyz="0 0 ${rear_shock_offset} "/>
+    <origin xyz="${wheelbase/2} 0 ${rear_shock_offset + chasisheight/2}"/>
   </joint>
 	<!-- rear axle -->
@@ -90,7 +90,7 @@
       dimz="${axlesize}" />
 	<joint name="base_link_to_rear_axle" type="fixed">
-    <parent link="chassis"/>
+    <parent link="base_link"/>
     <child link="rear_axle"/>
-    <origin xyz="${-wheelbase/2} 0 ${-chasisheight/2 - rear_shock_offset} "/>
+    <origin xyz="0 0 0"/>
   </joint>
 	<!-- right rear wheel -->
@@ -299,5 +299,5 @@
 		<material>Gazebo/Red</material>
 	</gazebo>
-	<joint name="back_to_left_arm" type="revolute">
+	<joint name="back_to_left_arm" type="fixed">
 		<axis xyz="0 -1 0"/>
     <limit effort="1000.0" lower="${liftmin}" upper="${liftmax}" velocity="0.5"/>
@@ -326,5 +326,5 @@
 		<material>Gazebo/Red</material>
 	</gazebo>
-	<joint name="back_to_right_arm" type="revolute">
+	<joint name="back_to_right_arm" type="fixed">
 		<axis xyz="0 -1 0"/>
     <limit effort="1000.0" lower="${liftmin}" upper="${liftmax}" velocity="0.5"/>
@@ -340,5 +340,5 @@
   </link>
 	<!-- lift front wall with arm -->
-	<joint name="left_arm_to_fork_assembly" type="revolute">
+	<joint name="left_arm_to_fork_assembly" type="fixed">
 		<axis xyz="0 -1 0"/>
     <limit effort="1000.0" lower="${liftmin}" upper="${liftmax}" velocity="0.5"/>
@@ -438,5 +438,5 @@
     </joint>
   </transmission>
-	<!-- Loader arm transmissions -->
+	<!-- Loader arm transmissions
 	<transmission name="left_arm_trans">
     <type>transmission_interface/SimpleTransmission</type>
@@ -466,8 +466,9 @@
     </joint>
   </transmission>
+-->
 	<!-- Specify Plugin for Gazebo-->
 	<gazebo>
     <plugin name="gazebo_ros_control" filename="libgazebo_ros_control.so">
-      <robotNamespace>/fitzroy</robotNamespace>
+      <robotNamespace>/</robotNamespace>
       <robotSimType>gazebo_ros_control/DefaultRobotHWSim</robotSimType>
       <legacyModeNS>true</legacyModeNS>
@@ -530,10 +531,10 @@
 	<!-- Camera -->
   <xacro:include filename="$(find fitzroy_description)/urdf/picam.urdf.xacro"/>
-  <picam parent="base_link" name="camera">
+  <picam parent="chassis" name="camera">
     <origin xyz="${-(wheelbase/2 + rackback)} 0 ${rackheight}" rpy="0 0 0"/>
   </picam>
 	<!-- Ultrasonic -->
   <xacro:include filename="$(find fitzroy_description)/urdf/ultrasonic_sensor.urdf.xacro"/>
-  <ultrasonic_sensor parent="base_link" name="ultrasonic">
+  <ultrasonic_sensor parent="chassis" name="ultrasonic">
     <origin xyz="${-(wheelbase/2 + rackback)} 0.020 ${rackheight}" rpy="0 0 0"/>
   </ultrasonic_sensor>

Commit message: Effort only i guess?

File: fitzroy_description/urdf/fitzroy.urdf.xacro (robot description, xacro)
@@ -58,7 +58,4 @@
 	<xacro:property name="propel_eff_limit" value="100000.0"/>
   <xacro:property name="propel_vel_limit" value="50.0"/>
-  <!-- Sensor Locations -->
-  <xacro:property name="gps_y" value="-0.02"/>
-  <xacro:property name="ranger_size" value="0.01"/>
 	<!-- base footprint to make everything work better -->
   <link name="base_footprint">
@@ -300,6 +297,6 @@
 	</gazebo>
 	<joint name="back_to_left_arm" type="fixed">
-		<axis xyz="0 -1 0"/>
-    <limit effort="1000.0" lower="${liftmin}" upper="${liftmax}" velocity="0.5"/>
+		<!--axis xyz="0 -1 0"/>
+    <limit effort="1000.0" lower="${liftmin}" upper="${liftmax}" velocity="0.5"/-->
     <parent link="chassis"/>
     <child link="left_arm"/>
@@ -327,6 +324,6 @@
 	</gazebo>
 	<joint name="back_to_right_arm" type="fixed">
-		<axis xyz="0 -1 0"/>
-    <limit effort="1000.0" lower="${liftmin}" upper="${liftmax}" velocity="0.5"/>
+		<!--axis xyz="0 -1 0"/>
+    <limit effort="1000.0" lower="${liftmin}" upper="${liftmax}" velocity="0.5"/-->
     <parent link="chassis"/>
     <child link="right_arm"/>
@@ -341,6 +338,6 @@
 	<!-- lift front wall with arm -->
 	<joint name="left_arm_to_fork_assembly" type="fixed">
-		<axis xyz="0 -1 0"/>
-    <limit effort="1000.0" lower="${liftmin}" upper="${liftmax}" velocity="0.5"/>
+		<!--axis xyz="0 -1 0"/>
+    <limit effort="1000.0" lower="${liftmin}" upper="${liftmax}" velocity="0.5"/-->
     <parent link="left_arm"/>
     <child link="fork_assembly"/>

File: fitzroy_description/urdf/fitzroy_common.urdf.xacro (robot description, xacro)
@@ -35,7 +35,7 @@
       <inertia ixx="${(1/12)*mass*(height*height) + (1 / 4)*mass*(rad*rad) }"
                ixy="0" ixz="0"
-               iyy="${(1/12)*mass*(height*height) + (1 / 4)*mass*(rad*rad) }"
+               iyy="${(1/2)* mass * (rad*rad)}"
                iyz="0"
-               izz="${(1/2)* mass * (rad*rad)}"/>
+               izz="${(1/12)*mass*(height*height) + (1 / 4)*mass*(rad*rad) }"/>
     </inertial>
   </xacro:macro>

Commit message: Added TF's for tof and us sensors to URDF. They are wrong, but at least they are present?

File: fitzroy_description/urdf/fitzroy.urdf.xacro (robot description, xacro)
@@ -510,7 +510,7 @@
   <joint name="imu_joint" type="fixed">
     <parent link="base_link"/>
-    <child link="imu_link"/>
-  </joint>
-	<link name="imu_link">
+    <child link="fitzroy_imu"/>
+  </joint>
+	<link name="fitzroy_imu">
 	</link>
 	<gazebo>
@@ -518,6 +518,6 @@
     <plugin name="imu_plugin" filename="libhector_gazebo_ros_imu.so">
         <alwaysOn>true</alwaysOn>
-        <bodyName>imu_link</bodyName>
-				<frameId>imu_link</frameId> <!-- 'frameId' not 'frameName'-->
+        <bodyName>fitzroy_imu</bodyName>
+				<frameId>fitzroy_imu</frameId> <!-- 'frameId' not 'frameName'-->
         <topicName>imu/data</topicName>
         <serviceName>imu/service</serviceName>
@@ -533,6 +533,21 @@
 	<!-- Ultrasonic -->
   <xacro:include filename="$(find fitzroy_description)/urdf/ultrasonic_sensor.urdf.xacro"/>
-  <ultrasonic_sensor parent="chassis" name="ultrasonic">
+  <ultrasonic_sensor parent="chassis" name="fitzroy_us1">
     <origin xyz="${-(wheelbase/2 + rackback)} 0.020 ${rackheight}" rpy="0 0 0"/>
   </ultrasonic_sensor>
+	<!-- Ultrasonic -->
+  <xacro:include filename="$(find fitzroy_description)/urdf/ultrasonic_sensor.urdf.xacro"/>
+  <ultrasonic_sensor parent="chassis" name="fitzroy_us2">
+    <origin xyz="${-(wheelbase/2 + rackback)} -0.020 ${rackheight}" rpy="0 0 0"/>
+  </ultrasonic_sensor>
+	<!-- TOF Rev -->
+  <xacro:include filename="$(find fitzroy_description)/urdf/ultrasonic_sensor.urdf.xacro"/>
+  <ultrasonic_sensor parent="chassis" name="fitzroy_tof1">
+    <origin xyz="${-(wheelbase/2 + rackback)} 0 ${rackheight - 0.02}" rpy="0 0 ${pi}"/>
+  </ultrasonic_sensor>
+	<!-- TOF Fwd -->
+  <xacro:include filename="$(find fitzroy_description)/urdf/ultrasonic_sensor.urdf.xacro"/>
+  <ultrasonic_sensor parent="chassis" name="fitzroy_tof2">
+    <origin xyz="${-(wheelbase/2 + rackback)} 0 ${rackheight - 0.02}" rpy="0 0 0"/>
+  </ultrasonic_sensor>
 </robot>

File: fitzroy_description/urdf/ultrasonic_sensor.urdf.xacro (robot description, xacro)
@@ -1,10 +1,4 @@
 <?xml version="1.0"?>
 <robot xmlns:xacro="http://www.ros.org/wiki/xacro">
-	<material name="ultrasonic_pcb_color">
-		<color rgba="0 0.6 0 1"/>
-	</material>
-	<material name="ultrasonic_speaker_color">
-		<color rgba="0.3 0.3 0.3 1"/>
-	</material>
   <xacro:macro name="ultrasonic_sensor" params="name parent *origin ros_topic:=ultrasonic_sensor update_rate:=15 min_range:=0.02 max_range:=4.0 field_of_view:=0.2617993878 ray_count:=10 resolution:=0.001 gaussian_noise:=0.010">
     <xacro:property name="dimx" value="0.015"/>
@@ -15,10 +9,16 @@
     <xacro:property name="speaker_spacing" value="0.027"/>
     <xacro:property name="speaker_diameter" value="0.016"/>
+		<material name="${name}_pcb_color">
+			<color rgba="0 0.6 0 1"/>
+		</material>
+		<material name="${name}_speaker_color">
+			<color rgba="0.3 0.3 0.3 1"/>
+		</material>
     <joint name="${name}_joint" type="fixed">
       <xacro:insert_block name="origin" />
       <parent link="${parent}"/>
-      <child link="${name}_link"/>
+      <child link="${name}"/>
     </joint>
-    <link name="${name}_link">
+    <link name="${name}">
       <visual>
         <origin xyz="${-dimx/2 + pcb_thickness/2} 0 0" rpy="0 0 0" />
@@ -26,5 +26,5 @@
           <box size="${pcb_thickness} ${dimy} ${dimz}" />
         </geometry>
-			  <material name="ultrasonic_pcb_color"/>
+			  <material name="${name}_pcb_color"/>
       </visual>
       <collision>
@@ -46,5 +46,5 @@
          https://answers.ros.org/question/154816/color-issue-with-urdf-and-multiple-visual-tags/ -->
     <joint name="${name}_speakers_joint" type="fixed">
-      <parent link="${name}_link"/>
+      <parent link="${name}"/>
       <child link="${name}_speakers_link"/>
     </joint>
@@ -56,5 +56,5 @@
           <cylinder length="${dimx*0.99}" radius="${speaker_diameter/2}"/>
         </geometry>
-			  <material name="ultrasonic_speaker_color"/>
+			  <material name="${name}_speaker_color"/>
       </visual>
       <visual>
@@ -64,5 +64,5 @@
           <cylinder length="${dimx*0.99}" radius="${speaker_diameter/2}"/>
         </geometry>
-			  <material name="ultrasonic_speaker_color"/>
+			  <material name="${name}_speaker_color"/>
       </visual>
       <visual>
@@ -71,8 +71,8 @@
           <box size="${pcb_thickness*2} ${pcb_thickness*5} ${pcb_thickness*2}" />
         </geometry>
-			  <material name="ultrasonic_speaker_color"/>
+			  <material name="${name}_speaker_color"/>
       </visual>
     </link>
-    <gazebo reference="${name}_link">
+    <gazebo reference="${name}">
       <sensor type="ray" name="${name}">
         <always_on>true</always_on>
@@ -104,5 +104,5 @@
           <gaussianNoise>${gaussian_noise}</gaussianNoise>
           <topicName>${ros_topic}</topicName>
-          <frameId>${name}_link</frameId>
+          <frameId>${name}</frameId>
         </plugin>
       </sensor>
